File: bringup.kicad_sch (KiCad schematic)
At the start: 1 part, among them U1 ADA4940-1ACPZ-R7

Commit message: feat: added Larry's goofy ahh + finished my schematic
Other:
- added sheet DAC (dac.kicad_sch)
Changed lines of the file:
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@@
+		)
+	)
+	(sheet
+		(at 179.07 90.17)
+		(size 12.7 11.43)
+		(exclude_from_sim no)
+		(in_bom yes)
+		(on_board yes)
+		(dnp no)
+		(fields_autoplaced yes)
+		(stroke
+			(width 0.1524)
+			(type solid)
+		)
+		(fill
+			(color 0 0 0 0.0000)
+		)
+		(property "Sheetname" "DAC"
+			(at 179.07 89.4584 0)
+			(effects
+				(font
+					(size 1.27 1.27)
+				)
+				(justify left bottom)
+			)
+		)
+		(property "Sheetfile" "dac.kicad_sch"
+			(at 179.07 102.1846 0)
+			(effects
+				(font
+					(size 1.27 1.27)
+				)
+				(justify left top)
+			)
+		)
+		(instances
+			(project "bringup"
+				(path "/5c7bcd8c-0d45-4448-8715-3709db3cee3b"
+					(page "2")
+				)
+			)
 		)
 	)

Commit message: fix: finished layout for bina mina
Parts:
- removed U1: ADA4940-1ACPZ-R7, CP_16_21_ADI, symbol 2025-04-06_00-22-58:ADA4940-1ACPZ-R7
Connections:
- no-connect marks 0 -> 7
Other:
- added sheet ADC (ADC.kicad_sch)
- sheet DAC ports: added DAC+, DAC-, Vout; removed none
Changed lines of the file:
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@@
 	(generator_version "9.0")
 	(paper "A4")
-	(symbol
-		(lib_id "2025-04-06_00-22-58:ADA4940-1ACPZ-R7")
-		(at 107.95 95.25 0)
-		(unit 1)
+	(no_connect
+		(at 118.11 71.12)
+	)
+	(no_connect
+		(at 199.39 69.85)
+	)
+	(no_connect
+		(at 199.39 66.04)
+	)
+	(no_connect
+		(at 158.75 69.85)
+	)
+	(no_connect
+		(at 118.11 67.31)
+	)
+	(no_connect
+		(at 158.75 66.04)
+	)
+	(no_connect
+		(at 130.81 68.58)
+	)
+	(sheet
+		(at 158.75 60.96)
+		(size 40.64 13.97)
 		(exclude_from_sim no)
 		(in_bom yes)
@@
 		(dnp no)
 		(fields_autoplaced yes)
-		(property "Reference" "U1"
-			(at 130.81 85.09 0)
-			(effects
-				(font
-					(size 1.524 1.524)
-				)
-			)
+		(stroke
+			(width 0.1524)
+			(type solid)
 		)
-		(property "Value" "ADA4940-1ACPZ-R7"
-			(at 130.81 87.63 0)
-			(effects
-				(font
-					(size 1.524 1.524)
-				)
-			)
+		(fill
+			(color 0 0 0 0.0000)
 		)
-		(property "Footprint" "CP_16_21_ADI"
-			(at 107.95 95.25 0)
-			(effects
-				(font
-					(size 1.27 1.27)
-					(italic yes)
-				)
-				(hide yes)
-			)
-		)
-		(property "Datasheet" "ADA4940-1ACPZ-R7"
-			(at 107.95 95.25 0)
-			(effects
-				(font
-					(size 1.27 1.27)
-					(italic yes)
-				)
-				(hide yes)
-			)
-		)
-		(property "Description" ""
-			(at 107.95 95.25 0)
+		(property "Sheetname" "ADC"
+			(at 158.75 60.2484 0)
 			(effects
 				(font
 					(size 1.27 1.27)
 				)
-				(hide yes)
+				(justify left bottom)
 			)
 		)
-		(pin "14"
+		(property "Sheetfile" "ADC.kicad_sch"
+			(at 158.75 75.5146 0)
+			(effects
+				(font
+					(size 1.27 1.27)
+				)
+				(justify left top)
+			)
 		)
-		(pin "11"
+		(pin "ADC_CHIP_OUT+" output
+			(at 199.39 69.85 0)
+			(effects
+				(font
+					(size 1.27 1.27)
+				)
+				(justify right)
+			)
 		)
-		(pin "13"
+		(pin "ADC_CHIP_OUT-" output
+			(at 199.39 66.04 0)
+			(effects
+				(font
+					(size 1.27 1.27)
+				)
+				(justify right)
+			)
 		)
-		(pin "12"
+		(pin "ADC_EXT_IN+" input
+			(at 158.75 69.85 180)
+			(effects
+				(font
+					(size 1.27 1.27)
+				)
+				(justify left)
+			)
 		)
-		(pin "9"
-		)
-		(pin "10"
-		)
-		(pin "17"
-		)
-		(pin "15"
-		)
-		(pin "5"
-		)
-		(pin "4"
-		)
-		(pin "6"
-		)
-		(pin "2"
-		)
-		(pin "7"
-		)
-		(pin "16"
-		)
-		(pin "8"
-		)
-		(pin "1"
-		)
-		(pin "3"
+		(pin "ADC_EXT_IN-" input
+			(at 158.75 66.04 180)
+			(effects
+				(font
+					(size 1.27 1.27)
+				)
+				(justify left)
+			)
 		)
 		(instances
-			(project ""
+			(project "bringup"
 				(path "/5c7bcd8c-0d45-4448-8715-3709db3cee3b"
-					(reference "U1")
-					(unit 1)
+					(page "3")
 				)
 			)
@@
 	)
 	(sheet
-		(at 179.07 90.17)
+		(at 118.11 63.5)
 		(size 12.7 11.43)
 		(exclude_from_sim no)
@@
 		)
 		(property "Sheetname" "DAC"
-			(at 179.07 89.4584 0)
+			(at 118.11 62.7884 0)
 			(effects
 				(font
@@
 		)
 		(property "Sheetfile" "dac.kicad_sch"
-			(at 179.07 102.1846 0)
+			(at 118.11 75.5146 0)
 			(effects
 				(font
@@
 			)
 		)
+		(pin "DAC+" input
+			(at 118.11 71.12 180)
+			(effects
+				(font
+					(size 1.27 1.27)
+				)
+				(justify left)
+			)
+		)
+		(pin "DAC-" input
+			(at 118.11 67.31 180)
+			(effects
+				(font
+					(size 1.27 1.27)
+				)
+				(justify left)
+			)
+		)
+		(pin "Vout" output
+			(at 130.81 68.58 0)
+			(effects
+				(font
+					(size 1.27 1.27)
+				)
+				(justify right)
+			)
+		)
