File: dac.kicad_sch (KiCad schematic)
At the start: 9 parts

Commit message: feat: added Larry's goofy ahh + finished my schematic
Parts:
- removed U2: ~, symbol dac:THS3095
- added C1: 0.01uF, symbol Device:C
- added C2: 1uF, symbol Device:C
- added R10, R4: 0R, Resistor_SMD:R_0201_0603Metric, symbol Device:R
- added U3: ~, Package_TO_SOT_SMD:TSOT-23-6, symbol dac:LMV951
- R1, R2, R3, R5, R6, R7, R8, R9: footprint (none) -> Resistor_SMD:R_0201_0603Metric
Connections:
- net VDDA: now also C1.1, C2.1, R10.1, U3.6 (V+)
- net VSSA: now also C1.2, C2.2, R4.2, U3.2 (V-)
- net Vn: now also U3.4 (In-)
- net Vout: now also U3.1 (OUTPUT)
- net Vp: now also U3.3 (In+)
- new net SHUTDOWN: R10.2, R4.1, U3.5 (SHUTDOWN)

Commit message: fix: finished layout for bina mina
Parts:
- removed R10, R4: 0R, Resistor_SMD:R_0201_0603Metric, symbol Device:R
- C1, C2: footprint (none) -> Capacitor_SMD:C_0603_1608Metric
- R1, R2, R5: footprint Resistor_SMD:R_0201_0603Metric -> Resistor_SMD:R_0603_1608Metric
- R3: renamed from R6; footprint Resistor_SMD:R_0201_0603Metric -> Resistor_SMD:R_0603_1608Metric
- R4: renamed from R7; footprint Resistor_SMD:R_0201_0603Metric -> Resistor_SMD:R_0603_1608Metric
- R6: renamed from R8; footprint Resistor_SMD:R_0201_0603Metric -> Resistor_SMD:R_0603_1608Metric
- R7: renamed from R3; footprint Resistor_SMD:R_0201_0603Metric -> Resistor_SMD:R_0603_1608Metric
- R8: renamed from R9; footprint Resistor_SMD:R_0201_0603Metric -> Resistor_SMD:R_0603_1608Metric
- renumbered U3 to U1
Connections:
- net SHUTDOWN is gone; now on net VSSA: U1.5 (SHUTDOWN)
